Commit message: new URDF update

File: xArm_with_gripper.urdf (robot description, URDF)
Before this commit: robot xarm6_with_gripper, 15 links, 14 joints
Links:
- removed link left_finger
- removed link left_inner_knuckle
- removed link left_outer_knuckle
- removed link link1
- removed link link2
- removed link link3
- removed link link4
- removed link link5
- removed link link6
- removed link link_base
- removed link right_finger
- removed link right_inner_knuckle
- removed link right_outer_knuckle
- removed link world
- removed link xarm_gripper_base_link
- added link base_link, mass 0.1; collision mesh filename=package://xarm_description/meshes/stls/base.stl scale=1.0 1.0 1.0; visual mesh filename=package://xarm_description/meshes/stls/base.stl scale=1.0 1.0 1.0
- added link xarm_2_link, mass 0.1; collision mesh filename=package://xarm_description/meshes/stls/link2.stl scale=1.0 1.0 1.0; visual mesh filename=package://xarm_description/meshes/stls/link2.stl scale=1.0 1.0 1.0
- added link xarm_3_link, mass 0.1; collision mesh filename=package://xarm_description/meshes/stls/link3.stl scale=1.0 1.0 1.0; visual mesh filename=package://xarm_description/meshes/stls/link3.stl scale=1.0 1.0 1.0
- added link xarm_4_link, mass 0.1; collision mesh filename=package://xarm_description/meshes/stls/link4.stl scale=1.0 1.0 1.0; visual mesh filename=package://xarm_description/meshes/stls/link4.stl scale=1.0 1.0 1.0
- added link xarm_5_link, mass 0.1; collision mesh filename=package://xarm_description/meshes/stls/link5.stl scale=1.0 1.0 1.0; visual mesh filename=package://xarm_description/meshes/stls/link5.stl scale=1.0 1.0 1.0
- added link xarm_6_link, mass 0.1; collision mesh filename=package://xarm_description/meshes/stls/link6.stl scale=1.0 1.0 1.0; visual mesh filename=package://xarm_description/meshes/stls/link6.stl scale=1.0 1.0 1.0
Joints:
- removed joint drive_joint
- removed joint gripper_fix
- removed joint joint1
- removed joint joint2
- removed joint joint3
- removed joint joint4
- removed joint joint5
- removed joint joint6
- removed joint left_finger_joint
- removed joint left_inner_knuckle_joint
- removed joint right_finger_joint
- removed joint right_inner_knuckle_joint
- removed joint right_outer_knuckle_joint
- removed joint world_joint
- added joint xarm_2_joint: type revolute, parent xarm_3_link, child xarm_2_link, origin xyz=0 -0.001205 0.05306 rpy=0 0 0, axis 0 0 1, limit lower=-2.17494876 upper=1.63121157 effort=1000 velocity=1.0
- added joint xarm_3_joint: type revolute, parent xarm_4_link, child xarm_3_link, origin xyz=0 0.0 0.09825 rpy=0 0 0, axis 1 0 0, limit lower=-1.740612146 upper=1.86797401 effort=1000 velocity=1.0
- added joint xarm_4_joint: type revolute, parent xarm_5_link, child xarm_4_link, origin xyz=0 0.0 0.09765 rpy=0 0 0, axis 1 0 0, limit lower=-1.910427965 upper=1.910427965 effort=1000 velocity=1.0
- added joint xarm_5_joint: type revolute, parent xarm_6_link, child xarm_5_link, origin xyz=0 -0.0022 0.03195 rpy=0 0 0, axis 1 0 0, limit lower=-1.592023304 upper=1.86797401 effort=1000 velocity=1.0
- added joint xarm_6_joint: type revolute, parent base_link, child xarm_6_link, origin xyz=0 0.0 0.03603 rpy=0 0 0, axis 0 0 1, limit lower=-1.737238322 upper=1.79965407 effort=1000 velocity=1.0

Commit message: adjusted urdf and made script

File: xArm_with_gripper.urdf (robot description, URDF)
Before this commit: robot xarm, 6 links, 5 joints
Joints:
- joint xarm_2_joint: origin xyz=0 -0.001205 0.05306 rpy=0 0 0 -> xyz=0 -0.001205 0.135 rpy=0 0 0
- joint xarm_3_joint: origin xyz=0 0.0 0.09825 rpy=0 0 0 -> xyz=0 0.0 0.0944 rpy=0 0 0
- joint xarm_4_joint: origin xyz=0 0.0 0.09765 rpy=0 0 0 -> xyz=0 0.0 0.09824 rpy=0 0 0
